File: EDU-CIAA_Poncho_SumoRobot/UltraSonido.sch (KiCad schematic (older format))
At the start: 2 parts, among them P2 CONN_01X04, P6 CONN_01X04

Commit message: Reorganizo bibliotecas en esquemático y PCB. Reparo señal de 12V. Agrego Footprints. Coloco plantilla EDU-CIAA. Reparo asociación conector EDU-CIAA en sch y pcb.
Parts:
- P2, P6: footprint Pin_Headers:Pin_Header_Straight_1x04 -> sumo_robot:Pin_Header_Straight_1x04
Changed lines of the file:
@@
 EESchema Schematic File Version 2
-LIBS:PONCHO-CIAA-rescue
-LIBS:PONCHO-CIAA-cache
+LIBS:power
+LIBS:PonchoSumoRobot-cache
 EELAYER 25 0
 EELAYER END
@@
 F 0 "P2" H 3750 2600 50  0000 C CNN
 F 1 "CONN_01X04" V 3850 2350 50  0000 C CNN
-F 2 "Pin_Headers:Pin_Header_Straight_1x04" H 3750 2350 50  0001 C CNN
+F 2 "sumo_robot:Pin_Header_Straight_1x04" H 3750 2350 50  0001 C CNN
 F 3 "" H 3750 2350 50  0000 C CNN
 	1    3750 2350
@@
 F 0 "P6" H 5050 2600 50  0000 C CNN
 F 1 "CONN_01X04" V 5150 2350 50  0000 C CNN
-F 2 "Pin_Headers:Pin_Header_Straight_1x04" H 5050 2350 50  0001 C CNN
+F 2 "sumo_robot:Pin_Header_Straight_1x04" H 5050 2350 50  0001 C CNN
 F 3 "" H 5050 2350 50  0000 C CNN
 	1    5050 2350
