File: Arduino_Acceso_lab/pcb/shield.sch (KiCad schematic (older format))
At the start: 20 parts, among them K1 RELAY_C, K2 RELAY_C, P1 Power, P13 Timer RTC, P14 Sensor1, P15 Sensor2, P16 Luz1, P17 Luz2, P2 Analog, P3 Digital, P4 Digital, Q1 2N2222, Q2 2N2222

Commit message: Arduino Acceso Lab. Ultimas modificaciones al PCB.
Changed lines of the file:
@@
 EESchema Schematic File Version 2
+LIBS:shield-rescue
+LIBS:acceso
 LIBS:power
+LIBS:device
+LIBS:transistors
+LIBS:shield_arduino
+LIBS:conn
 LIBS:shield-cache
 EELAYER 25 0
@@
 $Descr A4 11693 8268
 encoding utf-8
-Sheet 1 1
+Sheet 1 2
 Title "shield sist. monitoreo"
 Date "lun. 30 mars 2015"
@@
 Connection ~ 3050 2500
 $Comp
-L +5V-RESCUE-shield #PWR01
+L +5V #PWR01
 U 1 1 579F3AFA
 P 2450 1925
@@
 $EndComp
 $Comp
-L +5V-RESCUE-shield #PWR02
+L +5V #PWR02
 U 1 1 579F3DB4
 P 4525 4775
@@
 $EndComp
 $Comp
-L +5V-RESCUE-shield #PWR03
+L +5V #PWR03
 U 1 1 579F3EEB
 P 7300 4775
@@
 $EndComp
 $Comp
-L +5V-RESCUE-shield #PWR04
+L +5V #PWR04
 U 1 1 579F3FFA
 P 8800 3900
@@
 $EndComp
 $Comp
-L +5V-RESCUE-shield #PWR05
+L +5V #PWR05
 U 1 1 579F40E1
 P 8800 3350
@@
 $EndComp
 $Comp
-L +5V-RESCUE-shield #PWR06
+L +5V #PWR06
 U 1 1 579F418C
 P 6975 775
@@
 $EndComp
 $Comp
-L GND-RESCUE-shield #PWR07
+L GND #PWR07
 U 1 1 579F4487
 P 2450 3975
@@
 $EndComp
 $Comp
-L GND-RESCUE-shield #PWR08
+L GND #PWR08
 U 1 1 579F4511
 P 6150 3975
@@
 $EndComp
 $Comp
-L GND-RESCUE-shield #PWR09
+L GND #PWR09
 U 1 1 579F4620
 P 4525 6250
@@
 $EndComp
 $Comp
-L GND-RESCUE-shield #PWR010
+L GND #PWR010
 U 1 1 579F46F3
 P 7300 6250
@@
 $EndComp
 $Comp
-L GND-RESCUE-shield #PWR011
+L GND #PWR011
 U 1 1 579F485C
 P 8025 3500
@@
 $EndComp
 $Comp
-L GND-RESCUE-shield #PWR012
+L GND #PWR012
 U 1 1 579F4943
 P 8025 3000
@@
 $EndComp
 $Comp
-L GND-RESCUE-shield #PWR013
+L GND #PWR013
 U 1 1 579F4A3E
 P 7350 1700
@@
 $EndComp
 $Comp
-L GND-RESCUE-shield #PWR014
+L GND #PWR014
 U 1 1 579F4B25
 P 8550 1750
@@
 $EndComp
 $Comp
-L GND-RESCUE-shield #PWR015
+L GND #PWR015
 U 1 1 579F4B6C
 P 8500 2425
