File: Arduino_Acceso_lab/pcb/shield.sch (KiCad schematic (older format))
At the start: 21 parts, among them K1 RELAY_C, K2 RELAY_C, P1 Power, P10 Analog, P11 Digital, P12 Digital, P13 Timer RTC, P14 Sensor1, P15 Sensor2, P16 Luz1, P17 Luz2, P2 Analog, P3 Digital, P4 Digital, P5 CONN_1, P6 CONN_1, P7 CONN_1, P8 CONN_1, P9 Power

Commit message: Ordenamiento de bibliotecas y footprints.
Parts:
- K1, K2: footprint Poncho_PLC:Relay_C -> huellas:Relay_C
- P1, P4: footprint Pin_Headers:Pin_Header_Straight_1x08_Pitch2.00mm -> (none)
- P10: footprint Pin_Headers:Pin_Header_Straight_1x06 -> huellas:Pin_Header_Straight_1x06
- P11: footprint Pin_Headers:Pin_Header_Straight_1x10 -> huellas:Pin_Header_Straight_1x10
- P12, P9: footprint Pin_Headers:Pin_Header_Straight_1x08 -> huellas:Pin_Header_Straight_1x08
- P13: footprint Socket_Strips:Socket_Strip_Straight_1x07 -> huellas:Socket_Strip_Straight_1x07
- P14, P15, P16, P17: footprint Poncho_PLC:BORNERA3 -> huellas:BORNERA3
- P2: footprint Pin_Headers:Pin_Header_Straight_1x06_Pitch2.00mm -> (none)
- P3: footprint Pin_Headers:Pin_Header_Straight_1x10_Pitch2.00mm -> (none)
- P5, P6, P7, P8: footprint Socket_Arduino_Uno:Arduino_1pin -> (none)
- SP1, SP2: footprint Buzzers_Beepers:Buzzer_12x9.5RM7.6 -> huellas:MagneticBuzzer_ProSignal_ABI-009-RC_RevA_25Oct2010
Changed lines of the file:
@@
 EESchema Schematic File Version 2
 LIBS:power
-LIBS:device
-LIBS:conn
-LIBS:74xgxx
-LIBS:74xx
-LIBS:ac-dc
-LIBS:actel
-LIBS:adc-dac
-LIBS:Altera
-LIBS:analog_devices
-LIBS:analog_switches
-LIBS:atmel
-LIBS:audio
-LIBS:brooktre
-LIBS:cmos4000
-LIBS:cmos_ieee
-LIBS:contrib
-LIBS:cypress
-LIBS:dc-dc
-LIBS:digital-audio
-LIBS:diode
-LIBS:display
-LIBS:dsp
-LIBS:elec-unifil
-LIBS:ESD_Protection
-LIBS:ftdi
-LIBS:gennum
-LIBS:graphic
-LIBS:hc11
-LIBS:intel
-LIBS:interface
-LIBS:ir
-LIBS:Lattice
-LIBS:linear
-LIBS:logo
-LIBS:maxim
-LIBS:memory
-LIBS:microchip
-LIBS:microchip_dspic33dsc
-LIBS:microchip_pic10mcu
-LIBS:microchip_pic12mcu
-LIBS:microchip_pic16mcu
-LIBS:microchip_pic18mcu
-LIBS:microchip_pic32mcu
-LIBS:microcontrollers
-LIBS:motor_drivers
-LIBS:motorola
-LIBS:msp430
-LIBS:nordicsemi
-LIBS:nxp_armmcu
-LIBS:onsemi
-LIBS:opto
-LIBS:Oscillators
-LIBS:philips
-LIBS:powerint
-LIBS:Power_Management
-LIBS:pspice
-LIBS:references
-LIBS:regul
-LIBS:relays
-LIBS:rfcom
-LIBS:sensors
-LIBS:silabs
-LIBS:siliconi
-LIBS:stm8
-LIBS:stm32
-LIBS:supertex
-LIBS:switches
-LIBS:texas
-LIBS:transf
-LIBS:transistors
-LIBS:ttl_ieee
-LIBS:valves
-LIBS:video
-LIBS:Xicor
-LIBS:xilinx
-LIBS:Zilog
-LIBS:st-microelectronics
-LIBS:Poncho_PLC
 LIBS:shield-cache
 EELAYER 25 0
@@
 F 0 "P1" V 9675 1875 60  0000 C CNN
 F 1 "Power" V 9775 1875 60  0000 C CNN
-F 2 "Pin_Headers:Pin_Header_Straight_1x08_Pitch2.00mm" H 9725 1875 60  0001 C CNN
+F 2 "" H 9725 1875 60  0001 C CNN
 F 3 "" H 9725 1875 60  0000 C CNN
 	1    9725 1875
@@
 F 0 "P2" V 9675 2675 60  0000 C CNN
 F 1 "Analog" V 9775 2675 60  0000 C CNN
-F 2 "Pin_Headers:Pin_Header_Straight_1x06_Pitch2.00mm" H 9725 2675 60  0001 C CNN
+F 2 "" H 9725 2675 60  0001 C CNN
 F 3 "" H 9725 2675 60  0000 C CNN
 	1    9725 2675
@@
 F 0 "P4" V 10000 2575 60  0000 C CNN
 F 1 "Digital" V 10100 2575 60  0000 C CNN
-F 2 "Pin_Headers:Pin_Header_Straight_1x08_Pitch2.00mm" H 10050 2575 60  0001 C CNN
+F 2 "" H 10050 2575 60  0001 C CNN
 F 3 "" H 10050 2575 60  0000 C CNN
 	1    10050 2575
@@
 F 0 "P3" V 10000 1575 60  0000 C CNN
 F 1 "Digital" V 10100 1575 60  0000 C CNN
-F 2 "Pin_Headers:Pin_Header_Straight_1x10_Pitch2.00mm" H 10050 1575 60  0001 C CNN
+F 2 "" H 10050 1575 60  0001 C CNN
 F 3 "" H 10050 1575 60  0000 C CNN
 	1    10050 1575
@@
 F 0 "P5" H 10955 650 40  0000 L CNN
 F 1 "CONN_1" H 10875 705 30  0001 C CNN
-F 2 "Socket_Arduino_Uno:Arduino_1pin" H 10875 650 60  0001 C CNN
+F 2 "" H 10875 650 60  0001 C CNN
 F 3 "" H 10875 650 60  0000 C CNN
 	1    10875 650
@@
 F 0 "P6" H 11030 650 40  0000 L CNN
 F 1 "CONN_1" H 10950 705 30  0001 C CNN
-F 2 "Socket_Arduino_Uno:Arduino_1pin" H 10950 650 60  0001 C CNN
+F 2 "" H 10950 650 60  0001 C CNN
 F 3 "" H 10950 650 60  0000 C CNN
 	1    10950 650
@@
 F 0 "P7" H 11105 650 40  0000 L CNN
 F 1 "CONN_1" H 11025 705 30  0001 C CNN
-F 2 "Socket_Arduino_Uno:Arduino_1pin" H 11025 650 60  0001 C CNN
+F 2 "" H 11025 650 60  0001 C CNN
 F 3 "" H 11025 650 60  0000 C CNN
 	1    11025 650
@@
 F 0 "P8" H 11180 650 40  0000 L CNN
 F 1 "CONN_1" H 11100 705 30  0001 C CNN
-F 2 "Socket_Arduino_Uno:Arduino_1pin" H 11100 650 60  0001 C CNN
+F 2 "" H 11100 650 60  0001 C CNN
 F 3 "" H 11100 650 60  0000 C CNN
 	1    11100 650
@@
 F 0 "P9" V 3300 2425 60  0000 C CNN
 F 1 "Power" V 3400 2425 60  0000 C CNN
-F 2 "Pin_Headers:Pin_Header_Straight_1x08" H 3350 2425 60  0001 C CNN
+F 2 "huellas:Pin_Header_Straight_1x08" H 3350 2425 60  0001 C CNN
 F 3 "" H 3350 2425 60  0000 C CNN
 	1    3350 2425
@@
 F 0 "P10" V 3300 3225 60  0000 C CNN
 F 1 "Analog" V 3400 3225 60  0000 C CNN
-F 2 "Pin_Headers:Pin_Header_Straight_1x06" H 3350 3225 60  0001 C CNN
+F 2 "huellas:Pin_Header_Straight_1x06" H 3350 3225 60  0001 C CNN
 F 3 "" H 3350 3225 60  0000 C CNN
 	1    3350 3225
@@
 F 0 "P12" V 3625 3125 60  0000 C CNN
 F 1 "Digital" V 3725 3125 60  0000 C CNN
-F 2 "Pin_Headers:Pin_Header_Straight_1x08" H 3675 3125 60  0001 C CNN
+F 2 "huellas:Pin_Header_Straight_1x08" H 3675 3125 60  0001 C CNN
 F 3 "" H 3675 3125 60  0000 C CNN
 	1    3675 3125
@@
 F 0 "P11" V 3625 2125 60  0000 C CNN
 F 1 "Digital" V 3725 2125 60  0000 C CNN
-F 2 "Pin_Headers:Pin_Header_Straight_1x10" H 3675 2125 60  0001 C CNN
+F 2 "huellas:Pin_Header_Straight_1x10" H 3675 2125 60  0001 C CNN
 F 3 "" H 3675 2125 60  0000 C CNN
 	1    3675 2125
@@
 F 0 "P14" H 1975 5975 50  0000 C CNN
 F 1 "Sensor1" V 2075 5775 50  0000 C CNN
-F 2 "Poncho_PLC:BORNERA3" H 1975 5775 50  0001 C CNN
+F 2 "huellas:BORNERA3" H 1975 5775 50  0001 C CNN
 F 3 "" H 1975 5775 50  0000 C CNN
 	1    1975 5775
@@
 F 0 "P15" H 1975 5500 50  0000 C CNN
 F 1 "Sensor2" V 2075 5300 50  0000 C CNN
-F 2 "Poncho_PLC:BORNERA3" H 1975 5300 50  0001 C CNN
+F 2 "huellas:BORNERA3" H 1975 5300 50  0001 C CNN
 F 3 "" H 1975 5300 50  0000 C CNN
 	1    1975 5300
@@
 F 0 "P13" H 2000 4925 50  0000 C CNN
 F 1 "Timer RTC" V 2100 4525 50  0000 C CNN
-F 2 "Socket_Strips:Socket_Strip_Straight_1x07" H 2000 4525 50  0001 C CNN
+F 2 "huellas:Socket_Strip_Straight_1x07" H 2000 4525 50  0001 C CNN
 F 3 "" H 2000 4525 50  0000 C CNN
 	1    2000 4525
@@
 F 0 "P16" H 4600 6500 50  0000 C CNN
 F 1 "Luz1" V 4700 6300 50  0000 C CNN
-F 2 "Poncho_PLC:BORNERA3" H 4600 6300 50  0001 C CNN
+F 2 "huellas:BORNERA3" H 4600 6300 50  0001 C CNN
 F 3 "" H 4600 6300 50  0000 C CNN
 	1    4600 6300
@@
 F 0 "P17" H 6375 6450 50  0000 C CNN
 F 1 "Luz2" V 6475 6250 50  0000 C CNN
-F 2 "Poncho_PLC:BORNERA3" H 6375 6250 50  0001 C CNN
+F 2 "huellas:BORNERA3" H 6375 6250 50  0001 C CNN
 F 3 "" H 6375 6250 50  0000 C CNN
 	1    6375 6250
@@
 F 0 "K1" V 4425 5300 60  0000 C CNN
 F 1 "RELAY_C" V 4425 4815 60  0000 C CNN
-F 2 "Poncho_PLC:Relay_C" H 4425 5050 60  0001 C CNN
+F 2 "huellas:Relay_C" H 4425 5050 60  0001 C CNN
 F 3 "" H 4425 5050 60  0000 C CNN
 	1    4425 5050
@@
 F 0 "K2" V 6200 5300 60  0000 C CNN
 F 1 "RELAY_C" V 6200 4815 60  0000 C CNN
-F 2 "Poncho_PLC:Relay_C" H 6200 5050 60  0001 C CNN
+F 2 "huellas:Relay_C" H 6200 5050 60  0001 C CNN
 F 3 "" H 6200 5050 60  0000 C CNN
 	1    6200 5050
@@
 F 0 "SP2" H 8800 4700 50  0000 C CNN
 F 1 "buzzer1" H 8800 4200 50  0000 C CNN
-F 2 "Buzzers_Beepers:Buzzer_12x9.5RM7.6" H 8900 4450 50  0001 C CNN
+F 2 "huellas:MagneticBuzzer_ProSignal_ABI-009-RC_RevA_25Oct2010" H 8900 4450 50  0001 C CNN
 F 3 "" H 8900 4450 50  0000 C CNN
 	1    8900 4450
@@
 F 0 "SP1" H 8775 5625 50  0000 C CNN
 F 1 "buzzer2" H 8775 5125 50  0000 C CNN
-F 2 "Buzzers_Beepers:Buzzer_12x9.5RM7.6" H 8875 5375 50  0001 C CNN
+F 2 "huellas:MagneticBuzzer_ProSignal_ABI-009-RC_RevA_25Oct2010" H 8875 5375 50  0001 C CNN
 F 3 "" H 8875 5375 50  0000 C CNN
 	1    8875 5375

Commit message: Modificaciones propuestas al esquemático de acceso_lab.
Connections:
- net labels added: GND
- wire segments 131 -> 136
Other:
- note added: "EL OTRO ASI COMO ESTE"
- moved on the sheet: K1, K2, P10, P11, P12, P13, P14, P15, P16, P17, P9

Commit message: Corrijo faltante de +5V y quito biblioteca power del Acceso_lab.
Connections:
- net labels added: +5V
- wire segments 136 -> 133
Other:
- note added: "ACA TE PUSE UN +5V\n"
- note added: "ACA TE PUSE UNA TIERRA"
Changed lines of the file:
@@
 Text Label 3325 2875 1    60   ~ 0
 3.3v
-Text Label 3200 2875 1    60   ~ 0
-5v
 $Comp
 L CONN_01X03 P14
@@
 	9050 1925 9375 1925
 Wire Wire Line
-	9300 2025 9300 2125
-Wire Wire Line
-	9300 2125 9300 3150
+	9300 2025 9300 3150
 Wire Wire Line
 	8600 1725 9375 1725
@@
 	4550 2750 5525 2750
 Wire Wire Line
-	4550 2650 5275 2650
+	5475 2650 4550 2650
 Wire Wire Line
 	3325 3350 3525 3350
@@
 	3200 3450 3525 3450
 Wire Wire Line
-	3450 3550 3450 3650
-Wire Wire Line
-	3450 3650 3450 4725
+	3450 3550 3450 4725
 Wire Wire Line
 	2750 3250 3525 3250
@@
 	3450 3150 3525 3150
 Wire Wire Line
-	3200 2875 3200 3450
+	3200 2700 3200 3450
 Wire Wire Line
 	3075 2875 3075 3750
@@
 	5525 2750 5525 2275
 Wire Wire Line
-	5275 2625 5475 2625
-Wire Wire Line
-	5475 2625 5475 2175
+	5475 2175 5475 2650
 Wire Wire Line
 	4650 6125 4650 6275
@@
 Text Notes 4050 6825 0    60   ~ 0
 EL OTRO ASI COMO ESTE
+$Comp
+L +5V #PWR?
+U 1 1 57915C02
+P 3200 2700
+F 0 "#PWR?" H 3200 2550 50  0001 C CNN
+F 1 "+5V" H 3200 2840 50  0000 C CNN
+F 2 "" H 3200 2700 50  0000 C CNN
+F 3 "" H 3200 2700 50  0000 C CNN
+	1    3200 2700
+	1    0    0    -1
+$EndComp
+Text Notes 2675 2475 0    60   ~ 0
+ACA TE PUSE UN +5V\n
+Text Notes 6350 3775 0    60   ~ 0
+ACA TE PUSE UNA TIERRA
 $EndSCHEMATC

Commit message: Actualizo pcb del Arduino Acceso lab.
Parts:
- removed P10: Analog, huellas:Pin_Header_Straight_1x06, symbol CONN_6
- removed P11: Digital, huellas:Pin_Header_Straight_1x10, symbol CONN_10
- removed P12: Digital, huellas:Pin_Header_Straight_1x08, symbol CONN_8
- removed P5, P6, P7, P8: CONN_1, symbol CONN_1
- removed P9: Power, huellas:Pin_Header_Straight_1x08, symbol CONN_8
- added D1, D2: 1N4001, Diodes_ThroughHole:Diode_DO-35_SOD27_Horizontal_RM10, symbol D
- added Q1, Q2: 2N2222, kicad:TO92-L21, symbol Q_NPN_EBC
- added R1, R2: 1K, Resistors_ThroughHole:Resistor_Horizontal_RM7mm, symbol R
- added SH1: ARDUINO_as_UNO, SHIELD_ARDUINO:ARDUINO_as_UNO_R3, symbol ARDUINO_as_UNO
- K1, K2: footprint huellas:Relay_C -> Poncho_PLC:Relay_C
- P1, P4: footprint (none) -> Socket_Strips:Socket_Strip_Straight_1x08
- P2: footprint (none) -> Socket_Strips:Socket_Strip_Straight_1x06
- P3: footprint (none) -> Socket_Strips:Socket_Strip_Straight_1x10
- SP1, SP2: footprint huellas:MagneticBuzzer_ProSignal_ABI-009-RC_RevA_25Oct2010 -> Connect:PINHEAD1-2
Connections:
- net labels removed: 0(Rx), 1(Tx), 10(**/SS), 11(**/MOSI), 12(MISO), 13(SCK), 2, 3.3v, 4, 5(**), 5v, 6(**), 7, 8, 9(**), A0, A1, A2, A4(SDA), A5(SCL), AREF, IOREF, Reset, Vin, gnd
- wire segments 133 -> 161
- no-connect marks 9 -> 4
Other:
- note removed: "ACA TE PUSE UN +5V\n"
- note removed: "ACA TE PUSE UNA TIERRA"
- note removed: "EL OTRO ASI COMO ESTE"
- note removed: "Holes"
- note removed: "Shield for Arduino that uses\nthe same pin disposition\nlike "Uno" board Rev 3."
- moved on the sheet: K1, K2, P13, P14, P15, P16, P17

Commit message: Agrego mejoras al shield para acceso lab.
Parts:
- removed SP1: buzzer2, Connect:PINHEAD1-2, symbol SPEAKER
- removed SP2: buzzer1, Connect:PINHEAD1-2, symbol SPEAKER
- added C1, C2: CP1, Capacitors_ThroughHole:C_Rect_L7.5_W6.5_P5, symbol CP1
- added C3: C, Capacitors_ThroughHole:C_Rect_L7.5_W6.5_P5, symbol C
- added D3: D, Diodes_ThroughHole:Diode_DO-35_SOD27_Horizontal_RM10, symbol D
- added D4: LED, LEDs:LED-3MM, symbol LED
- added L1: INDUCTOR, Inductors:INDUCTOR_V, symbol INDUCTOR
- added P5: modulo esp8266, Socket_Strips:Socket_Strip_Straight_2x04, symbol CONN_02X04
- added P6: fuente, Connect:PINHEAD1-2, symbol CONN_01X02
- added P7: buzzer 1, Pin_Headers:Pin_Header_Straight_1x02, symbol CONN_01X02
- added P8: buzzer 2, Pin_Headers:Pin_Header_Straight_1x02, symbol CONN_01X02
- added R3, R4, R5, R6, R7: R, Resistors_ThroughHole:Resistor_Horizontal_RM7mm, symbol R
- added U1: LM2576, TO_SOT_Packages_THT:Pentawatt_Neutral_Staggered_Verical_TO220-5-T05D, symbol LM2576
- SH1: symbol ARDUINO_as_UNO -> ARDUINO_as_UNO-RESCUE-shield
- renumbered P14 to P10, P15 to P11, P16 to P12, P17 to P13, P13 to P9
Connections:
- net labels added: +3.3VP, +5P, GNDD, VCC, rx-wifi, tx-wifi
- net labels removed: +5V, GND
- wire segments 161 -> 208
- no-connect marks 4 -> 7
Other:
- moved on the sheet: D1, D2, K1, K2, P1, P10, P11, P12, P13, P9, Q1, Q2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
