File: Arduino_SumoRobot/sumo.sch (KiCad schematic (older format))
At the start: 77 parts, among them IC1 40106D, K1 RELAY_C, K2 RELAY_C, K3 RELAY_C, K4 RELAY_C, P1 Power, P10 CONN_01X04, P11 CONN_01X04, P12 CONN_BATERIA12V, P13 CONN_01X02, P14 CONN_01X02, P17 CONN_01X02, P18 CONN_01X02, P19 CONN_02X16, P2 Analog, P3 Digital, P4 Digital, P5 CONN_1, P6 CONN_1, P7 CONN_1, P8 CONN_1, P9 CONN_01X06, Q1 S8050, Q2 S8050, Q3 S8050, Q4 S8050, U1 LM2576

Commit message: Arduino Sumo. Cambio todos los leds a 3mm porque había una mezcla.
Parts:
- D10, D11, D6, D7, D8, D9, Rojo1: footprint huellas:LED-5MM -> huellas:led-LED3MM; symbol LED -> LED3MM
Connections:
- net 2: now also D7.K (C); no longer D7.1 (K)
- net 3(**): now also D6.K (C); no longer D6.1 (K)
- net VCC: now also Rojo1.A; no longer Rojo1.2 (A)
- net at IC1.12 (O), P3.1 (P1): now also D10.K (C); no longer D10.1 (K)
- net at IC1.10 (O), P3.2 (P2): now also D11.K (C); no longer D11.1 (K)
- net at IC1.6 (O), P3.5 (P5): now also D8.K (C); no longer D8.1 (K)
- net at IC1.8 (O), P3.6 (P6): now also D9.K (C); no longer D9.1 (K)
- net at R18.2: now also D7.A; no longer D7.2 (A)
- net at R19.2: now also D8.A; no longer D8.2 (A)
- net at R20.2: now also D9.A; no longer D9.2 (A)
- net at R17.2: now also D6.A; no longer D6.2 (A)
- net at R21.1: now also Rojo1.K (C); no longer Rojo1.1 (K)
- net at R26.2: now also D11.A; no longer D11.2 (A)
- net at R27.2: now also D10.A; no longer D10.2 (A)
Changed lines of the file:
@@
 $EndComp
 $Comp
-L LED Rojo1
+L LED3MM Rojo1
 U 1 1 580AFB0F
-P 8700 1100
-F 0 "Rojo1" H 8700 1200 50  0000 C CNN
-F 1 "LED" H 8700 1000 50  0000 C CNN
-F 2 "huellas:LED-5MM" H 8700 1100 50  0001 C CNN
-F 3 "" H 8700 1100 50  0000 C CNN
-	1    8700 1100
-	0    -1   -1   0
+P 8700 1075
+F 0 "Rojo1" H 8700 1175 50  0000 C CNN
+F 1 "LED" H 8550 825 50  0000 C CNN
+F 2 "huellas:led-LED3MM" H 8700 1075 50  0001 C CNN
+F 3 "" H 8700 1075 50  0000 C CNN
+	1    8700 1075
+	1    0    0    -1
 $EndComp
 $Comp
@@
 $EndComp
 $Comp
-L LED D8
+L LED3MM D8
 U 1 1 58173729
-P 4225 1400
-F 0 "D8" H 4425 1450 50  0000 C CNN
-F 1 "LED" H 4000 1450 50  0000 C CNN
-F 2 "huellas:LED-5MM" H 4225 1400 50  0001 C CNN
-F 3 "" H 4225 1400 50  0000 C CNN
-	1    4225 1400
-	0    -1   -1   0
-$EndComp
-$Comp
-L LED D9
+P 4225 1350
+F 0 "D8" V 4175 1475 50  0000 C CNN
+F 1 "LED" V 4175 1075 50  0000 C CNN
+F 2 "huellas:led-LED3MM" H 4225 1350 50  0001 C CNN
+F 3 "" H 4225 1350 50  0000 C CNN
+	1    4225 1350
+	1    0    0    -1
+$EndComp
+$Comp
+L LED3MM D9
 U 1 1 581746E0
-P 4050 1400
-F 0 "D9" H 4250 1450 50  0000 C CNN
-F 1 "LED" H 3825 1450 50  0000 C CNN
-F 2 "huellas:LED-5MM" H 4050 1400 50  0001 C CNN
-F 3 "" H 4050 1400 50  0000 C CNN
-	1    4050 1400
-	0    -1   -1   0
-$EndComp
-$Comp
-L LED D7
+P 4050 1350
+F 0 "D9" V 4000 1475 50  0000 C CNN
+F 1 "LED" V 4000 1075 50  0000 C CNN
+F 2 "huellas:led-LED3MM" H 4050 1350 50  0001 C CNN
+F 3 "" H 4050 1350 50  0000 C CNN
+	1    4050 1350
+	1    0    0    -1
+$EndComp
+$Comp
+L LED3MM D7
 U 1 1 58175877
-P 4400 1400
-F 0 "D7" H 4600 1475 50  0000 C CNN
-F 1 "LED" H 4175 1450 50  0000 C CNN
-F 2 "huellas:LED-5MM" H 4400 1400 50  0001 C CNN
-F 3 "" H 4400 1400 50  0000 C CNN
-	1    4400 1400
-	0    -1   -1   0
-$EndComp
-$Comp
-L LED D6
+P 4400 1350
+F 0 "D7" V 4350 1475 50  0000 C CNN
+F 1 "LED" V 4350 1075 50  0000 C CNN
+F 2 "huellas:led-LED3MM" H 4400 1350 50  0001 C CNN
+F 3 "" H 4400 1350 50  0000 C CNN
+	1    4400 1350
+	1    0    0    -1
+$EndComp
+$Comp
+L LED3MM D6
 U 1 1 581759E7
-P 4575 1400
-F 0 "D6" H 4775 1475 50  0000 C CNN
-F 1 "LED" H 4350 1450 50  0000 C CNN
-F 2 "huellas:LED-5MM" H 4575 1400 50  0001 C CNN
-F 3 "" H 4575 1400 50  0000 C CNN
-	1    4575 1400
-	0    -1   -1   0
+P 4575 1350
+F 0 "D6" V 4525 1475 50  0000 C CNN
+F 1 "LED" V 4525 1075 50  0000 C CNN
+F 2 "huellas:led-LED3MM" H 4575 1350 50  0001 C CNN
+F 3 "" H 4575 1350 50  0000 C CNN
+	1    4575 1350
+	1    0    0    -1
 $EndComp
 $Comp
@@
 $EndComp
 $Comp
-L LED D10
+L LED3MM D10
 U 1 1 5819BAC7
-P 3000 4425
-F 0 "D10" H 3000 4525 50  0000 C CNN
-F 1 "LED" H 3000 4325 50  0000 C CNN
-F 2 "huellas:LED-5MM" H 2925 4775 50  0001 C CNN
-F 3 "" H 3000 4425 50  0000 C CNN
-	1    3000 4425
-	0    -1   -1   0
+P 3000 4375
+F 0 "D10" V 2900 4525 50  0000 C CNN
+F 1 "LED" V 3075 4525 50  0000 C CNN
+F 2 "huellas:led-LED3MM" H 2925 4725 50  0001 C CNN
+F 3 "" H 3000 4375 50  0000 C CNN
+	1    3000 4375
+	1    0    0    -1
 $EndComp
 $Comp
@@
 $EndComp
 $Comp
-L LED D11
+L LED3MM D11
 U 1 1 58122070
-P 2525 4425
-F 0 "D11" H 2525 4525 50  0000 C CNN
-F 1 "LED" H 2525 4325 50  0000 C CNN
-F 2 "huellas:LED-5MM" H 2525 4425 50  0001 C CNN
-F 3 "" H 2525 4425 50  0000 C CNN
-	1    2525 4425
-	0    -1   -1   0
+P 2525 4375
+F 0 "D11" V 2425 4475 50  0000 C CNN
+F 1 "LED" V 2600 4475 50  0000 C CNN
+F 2 "huellas:led-LED3MM" H 2525 4375 50  0001 C CNN
+F 3 "" H 2525 4375 50  0000 C CNN
+	1    2525 4375
+	1    0    0    -1
 $EndComp
 $Comp
@@
 	8125 1625 8125 1825
 Wire Wire Line
-	8700 1375 8700 1300
+	8700 1275 8700 1375
 Wire Wire Line
 	8125 750  8125 1325
@@
 	1275 3425 1125 3425
 Wire Wire Line
-	4575 1200 4575 1125
+	4575 1125 4575 1250
 Wire Wire Line
 	3900 1750 4575 1750
@@
 	4575 4450 5275 4450
 Wire Wire Line
-	4575 1600 4575 4450
+	4575 1550 4575 4450
 Connection ~ 4575 1750
 Wire Wire Line
 	5100 4550 4400 4550
 Wire Wire Line
-	4400 4550 4400 1600
+	4400 4550 4400 1550
 Connection ~ 4400 2350
 Wire Wire Line
 	4400 2350 3900 2350
 Wire Wire Line
-	4400 1200 4400 1125
+	4400 1125 4400 1250
 Wire Wire Line
 	4400 825  4400 700
@@
 	4225 700  4225 825
 Wire Wire Line
-	4225 1125 4225 1200
-Wire Wire Line
-	4225 1600 4225 5075
+	4225 1125 4225 1250
+Wire Wire Line
+	4225 1550 4225 5075
 Connection ~ 4225 3000
 Wire Wire Line
@@
 	4050 700  4050 825
 Wire Wire Line
-	4050 1125 4050 1200
-Wire Wire Line
-	4050 1600 4050 4925
+	4050 1125 4050 1250
+Wire Wire Line
+	4050 1550 4050 4925
 $Comp
 L GND-RESCUE-Arduino_As_Uno #PWR064
@@
 	1450 4350 1450 4275
 Wire Wire Line
-	3000 4625 3000 5350
+	3000 4575 3000 5350
 Connection ~ 3000 5350
 Wire Wire Line
-	2525 4625 2525 4700
+	2525 4575 2525 4700
 Connection ~ 2525 4700
 Wire Wire Line
@@
 $EndComp
 Wire Wire Line
-	2525 4225 2525 4150
-Wire Wire Line
-	3000 4225 3000 4150
+	2525 4150 2525 4275
+Wire Wire Line
+	3000 4150 3000 4275
 $Comp
 L +5V #PWR074
@@
 Wire Wire Line
 	5425 1250 5275 1250
+Wire Wire Line
+	8700 900  8700 975
 $EndSCHEMATC
