File: Arduino_SumoRobot/sumo.sch (KiCad schematic (older format))
At the start: 77 parts, among them IC1 40106D, K1 RELAY_C, K2 RELAY_C, K3 RELAY_C, K4 RELAY_C, P1 Power, P10 CONN_01X04, P11 CONN_01X04, P12 CONN_BATERIA12V, P13 CONN_01X02, P14 CONN_01X02, P17 CONN_01X02, P18 CONN_01X02, P19 CONN_02X16, P2 Analog, P3 Digital, P4 Digital, P5 CONN_1, P6 CONN_1, P7 CONN_1, P8 CONN_1, P9 CONN_01X06, Q1 S8050, Q2 S8050, Q3 S8050, Q4 S8050, U1 LM2576

Commit message: Agrego mejoras al Arduino Sumo Robot realizadas por el Grupo II de 2016.
Parts:
- C2: value C -> 100nF
- CP1: value CP1 -> 10uF
- CP2: value CP1 -> 100uF
- D1: value D -> 1N5819
- L1: value INDUCTOR -> 330uHy
- P19: footprint huellas:Pin_Header_Straight_2x16_Pitch2.00mm -> Pin_Headers:Pin_Header_Straight_2x16
- R17, R18, R19, R20, R21, R23, R24: value R -> 1K
Changed lines of the file:
@@
 LIBS:lm2576
 LIBS:dc-dc
+LIBS:sumo
 LIBS:sumo-cache
 EELAYER 25 0
@@
 P 4400 975
 F 0 "R18" V 4350 1175 50  0000 C CNN
-F 1 "R" V 4400 975 50  0000 C CNN
+F 1 "1K" V 4400 975 50  0000 C CNN
 F 2 "huellas:Resistor_Horizontal_RM7mm" V 5225 1000 50  0001 C CNN
 F 3 "" H 4400 975 50  0000 C CNN
@@
 P 4225 975
 F 0 "R19" V 4175 1175 50  0000 C CNN
-F 1 "R" V 4225 975 50  0000 C CNN
+F 1 "1K" V 4225 975 50  0000 C CNN
 F 2 "huellas:Resistor_Horizontal_RM7mm" V 5175 1450 50  0001 C CNN
 F 3 "" H 4225 975 50  0000 C CNN
@@
 P 4050 975
 F 0 "R20" V 4000 1175 50  0000 C CNN
-F 1 "R" V 4050 975 50  0000 C CNN
+F 1 "1K" V 4050 975 50  0000 C CNN
 F 2 "huellas:Resistor_Horizontal_RM7mm" V 4775 1150 50  0001 C CNN
 F 3 "" H 4050 975 50  0000 C CNN
@@
 P 4575 975
 F 0 "R17" V 4525 1175 50  0000 C CNN
-F 1 "R" V 4575 975 50  0000 C CNN
+F 1 "1K" V 4575 975 50  0000 C CNN
 F 2 "huellas:Resistor_Horizontal_RM7mm" V 5200 -900 50  0001 C CNN
 F 3 "" H 4575 975 50  0000 C CNN
@@
 P 7500 1225
 F 0 "L1" V 7450 1225 50  0000 C CNN
-F 1 "INDUCTOR" V 7350 1225 50  0000 C CNN
+F 1 "330uHy" V 7350 1225 50  0000 C CNN
 F 2 "huellas:INDUCTOR_V" H 7000 1475 50  0001 C CNN
 F 3 "" H 7500 1225 50  0000 C CNN
@@
 P 7150 1475
 F 0 "D1" H 7150 1575 50  0000 C CNN
-F 1 "D" H 7150 1375 50  0000 C CNN
+F 1 "1N5819" H 7150 1375 50  0000 C CNN
 F 2 "huellas:Diode_DO-41_SOD81_Horizontal_RM10" H 7150 1475 50  0001 C CNN
 F 3 "" H 7150 1475 50  0000 C CNN
@@
 P 8125 1475
 F 0 "C2" H 8150 1575 50  0000 L CNN
-F 1 "C" H 8150 1375 50  0000 L CNN
+F 1 "100nF" H 7900 1350 50  0000 L CNN
 F 2 "huellas:C_Rect_L7_W6_P5" H 8100 1475 50  0001 C CNN
 F 3 "" H 8125 1475 50  0000 C CNN
@@
 P 8700 1525
 F 0 "R21" V 8780 1525 50  0000 C CNN
-F 1 "R" V 8700 1525 50  0000 C CNN
+F 1 "1K" V 8700 1525 50  0000 C CNN
 F 2 "huellas:Resistor_Horizontal_RM7mm" V 8630 1525 50  0001 C CNN
 F 3 "" H 8700 1525 50  0000 C CNN
@@
 P 5425 1650
 F 0 "CP2" H 5450 1750 50  0000 L CNN
-F 1 "CP1" H 5450 1550 50  0000 L CNN
+F 1 "100uF" H 5450 1550 50  0000 L CNN
 F 2 "huellas:C_Radial_D6.3_L11.2_P2.5" H 7875 1625 50  0001 C CNN
 F 3 "" H 5425 1650 50  0000 C CNN
@@
 P 7875 1475
 F 0 "CP1" H 7900 1575 50  0000 L CNN
-F 1 "CP1" H 7900 1375 50  0000 L CNN
+F 1 "10uF" H 7650 1350 50  0000 L CNN
 F 2 "huellas:C_Radial_D6.3_L11.2_P2.5" H 7875 1475 50  0001 C CNN
 F 3 "" H 7875 1475 50  0000 C CNN
@@
 P 8350 1100
 F 0 "R23" V 8430 1100 50  0000 C CNN
-F 1 "R" V 8350 1100 50  0000 C CNN
+F 1 "1K" V 8350 1100 50  0000 C CNN
 F 2 "huellas:Resistor_Horizontal_RM7mm" V 8280 1100 50  0001 C CNN
 F 3 "" H 8350 1100 50  0000 C CNN
@@
 P 8350 1525
 F 0 "R24" V 8430 1525 50  0000 C CNN
-F 1 "R" V 8350 1525 50  0000 C CNN
+F 1 "1K" V 8350 1525 50  0000 C CNN
 F 2 "huellas:Resistor_Horizontal_RM7mm" V 8280 1525 50  0001 C CNN
 F 3 "" H 8350 1525 50  0000 C CNN
@@
 F 0 "P19" H 1525 3525 50  0000 C CNN
 F 1 "CONN_02X16" V 1525 2675 50  0000 C CNN
-F 2 "huellas:Pin_Header_Straight_2x16_Pitch2.00mm" H 1525 1575 50  0001 C CNN
+F 2 "Pin_Headers:Pin_Header_Straight_2x16" H 1525 1575 50  0001 C CNN
 F 3 "" H 1525 1575 50  0000 C CNN
 	1    1525 2675
