File: Arduino_Acceso_lab/pcb_expo/pcb.sch (KiCad schematic (older format))
At the start: 15 parts, among them P1 modulo wifi, P20 CONN_01X02, U1 LM2576

Commit message: Versión corregida por DJB del Shield Wifi para Arduini Mega.
Connections:
- net TXwifi is gone; now on net RXwifi: R2.2, SH1.18 (TXD1)
- net +9V: now also C2.1, C3.1, L1.2, R1.1, R4.1; no longer R4.2, R5.1
- net RXwifi: no longer P1.2 (P2), SH1.19 (RXD1)
- net at U1.4 (FB): now also R4.2, R5.1; no longer R4.1
- net 3.3 renamed +3.3VP
- new net TXwifi2: P1.2 (P2), SH1.19 (RXD1)
Changed lines of the file:
@@
 $EndComp
 Text Label 4425 3800 0    60   ~ 0
-RXwifi
+TXwifi2
 Text Label 9925 5475 0    60   ~ 0
-RXwifi
+TXwifi2
 $Comp
 L D D2
@@
 	1    0    0    -1
 $EndComp
-Text Label 1875 1800 0    60   ~ 0
-3.3
-Text Label 10175 5950 0    60   ~ 0
-3.3
 $Comp
 L GND-RESCUE-pcb #PWR05
@@
 $EndComp
 Text Label 8650 5775 2    60   ~ 0
-TXwifi
+RXwifi
 Text Label 4425 3700 0    60   ~ 0
-TXwifi
+RXwifi
 $Comp
 L +9V #PWR011
@@
 Connection ~ 10075 5800
 Wire Wire Line
-	10075 5950 10175 5950
+	10075 5950 10275 5950
 Wire Wire Line
 	4375 3800 4425 3800
@@
 Connection ~ 7625 1900
 Wire Wire Line
-	8525 1275 9475 1275
-Wire Wire Line
 	10500 1825 10500 1725
 Wire Wire Line
-	10175 1375 10175 1650
+	10175 1175 10175 1650
 Wire Wire Line
 	10500 1375 10500 1425
@@
 Wire Wire Line
 	9475 1775 9475 1850
-Wire Wire Line
-	9475 1275 9475 1475
-Wire Wire Line
-	9475 1825 9750 1825
-Wire Wire Line
-	9750 1825 9750 1150
 Connection ~ 9475 1825
 Wire Wire Line
@@
 Wire Wire Line
 	8550 2025 8550 1725
+Wire Wire Line
+	9475 1825 9225 1825
+Wire Wire Line
+	9225 1825 9225 1275
+Wire Wire Line
+	9225 1275 8525 1275
+Wire Wire Line
+	9475 1375 9475 1475
+Connection ~ 9475 1375
+Wire Wire Line
+	9750 1150 9750 1375
+Connection ~ 9750 1375
+$Comp
+L +3.3VP #PWR015
+U 1 1 58221380
+P 10275 5850
+F 0 "#PWR015" H 10425 5800 50  0001 C CNN
+F 1 "+3.3VP" H 10275 5950 50  0000 C CNN
+F 2 "" H 10275 5850 50  0000 C CNN
+F 3 "" H 10275 5850 50  0000 C CNN
+	1    10275 5850
+	1    0    0    -1
+$EndComp
+Wire Wire Line
+	10275 5950 10275 5850
+$Comp
+L +3.3VP #PWR016
+U 1 1 58221527
+P 1875 1225
+F 0 "#PWR016" H 2025 1175 50  0001 C CNN
+F 1 "+3.3VP" H 1875 1325 50  0000 C CNN
+F 2 "" H 1875 1225 50  0000 C CNN
+F 3 "" H 1875 1225 50  0000 C CNN
+	1    1875 1225
+	1    0    0    -1
+$EndComp
+Wire Wire Line
+	1875 1800 1875 1225
+$Comp
+L PWR_FLAG #FLG017
+U 1 1 58221C33
+P 6050 1825
+F 0 "#FLG017" H 6050 1920 50  0001 C CNN
+F 1 "PWR_FLAG" H 6050 2005 50  0000 C CNN
+F 2 "" H 6050 1825 50  0000 C CNN
+F 3 "" H 6050 1825 50  0000 C CNN
+	1    6050 1825
+	1    0    0    -1
+$EndComp
+Wire Wire Line
+	6050 1825 6050 1875
+Wire Wire Line
+	6050 1875 6375 1875
+Connection ~ 6375 1875
+$Comp
+L PWR_FLAG #FLG018
+U 1 1 582224EA
+P 1525 1300
+F 0 "#FLG018" H 1525 1395 50  0001 C CNN
+F 1 "PWR_FLAG" H 1525 1480 50  0000 C CNN
+F 2 "" H 1525 1300 50  0000 C CNN
+F 3 "" H 1525 1300 50  0000 C CNN
+	1    1525 1300
+	1    0    0    -1
+$EndComp
+Wire Wire Line
+	1875 1425 1525 1425
+Wire Wire Line
+	1525 1425 1525 1300
+Connection ~ 1875 1425
+$Comp
+L PWR_FLAG #FLG019
+U 1 1 58222672
+P 10175 1175
+F 0 "#FLG019" H 10175 1270 50  0001 C CNN
+F 1 "PWR_FLAG" H 10175 1355 50  0000 C CNN
+F 2 "" H 10175 1175 50  0000 C CNN
+F 3 "" H 10175 1175 50  0000 C CNN
+	1    10175 1175
+	1    0    0    -1
+$EndComp
 $EndSCHEMATC
